File: PM5644_Mainboard.sch (KiCad schematic (older format))
At the start: 15 parts, among them U101 27C4001, U102 74HC574, U109 27C4001, U111 74HC153, U14 74HC138, U31 74HC574, U32 74HC574, U33 74HC574, U34 74HC574, U35 74HC574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

Commit message: Updated
Connections:
- wire segments 287 -> 288
Changed lines of the file:
@@
 Connection ~ 16800 3400
 Wire Wire Line
-	16025 3200 16275 3200
-Text Label 16100 3200 0    50   ~ 0
+	16025 3100 16275 3100
+Text Label 16100 3100 0    50   ~ 0
 A16
 Wire Wire Line
@@
 	11000 3000 11225 3000
 Entry Wire Line
-	16275 3200 16375 3100
-Wire Bus Line
-	16375 3100 16375 1250
-Wire Bus Line
-	14600 1250 16375 1250
+	16275 3100 16375 3000
 Wire Wire Line
 	12225 2500 12475 2500
@@
 Entry Wire Line
 	16525 2500 16625 2600
-Wire Bus Line
-	16525 1250 16375 1250
-Connection ~ 16375 1250
 Text Notes 8400 1000 0    50   ~ 0
 TODO:\nCHECK FOR GROUNDED PINS ON PALS\nCHECK FOR OPEN PINS ON PALS
@@
 Connection ~ 7300 1250
 Wire Bus Line
+	14600 1250 16375 1250
+Wire Bus Line
+	16375 3000 16375 1250
+Connection ~ 16375 1250
+Wire Bus Line
+	16375 1250 16525 1250
+Wire Wire Line
+	16025 3300 16250 3300
+Wire Bus Line
 	4000 4325 4000 5650
 Wire Bus Line
@@
 Wire Bus Line
 	1000 4225 1000 6750
+Text Label 16100 3300 0    50   ~ 0
+P5
 $EndSCHEMATC
